File: BussBar.sch (KiCad schematic (older format))
At the start: 12 parts, among them J1 INPUT POWER, J2 Conn_02x05_Odd_Even, J3 Conn_02x05_Odd_Even, J4 Conn_02x05_Odd_Even, J5 Conn_02x05_Odd_Even, J6 Conn_02x05_Odd_Even, J7 Conn_02x05_Odd_Even

Commit message: V0.0.1 Chematic and PCB  - Initial to routing
Parts:
- added unit 2 of ON/OFF1
- ON/OFF1: symbol Switch:SW_DPST -> Switch:SW_DPDT_x2
Connections:
- net +12V: now also ON/OFF1.5 (B); no longer ON/OFF1.1
- net +12s: now also ON/OFF1.4 (A); no longer ON/OFF1.2
- net -12V: now also ON/OFF1.2 (B); no longer ON/OFF1.3
- net -12s: now also ON/OFF1.1 (A); no longer ON/OFF1.4
- net GND: now also J2.3 (Pin_3), J2.5 (Pin_5), J2.7 (Pin_7), J3.3 (Pin_3), J3.5 (Pin_5), J3.7 (Pin_7), J4.3 (Pin_3), J4.5 (Pin_5), J4.7 (Pin_7), J5.3 (Pin_3), J5.5 (Pin_5), J5.7 (Pin_7), J6.3 (Pin_3), J6.5 (Pin_5), J6.7 (Pin_7), J7.3 (Pin_3), J7.5 (Pin_5), J7.7 (Pin_7)
Changed lines of the file:
@@
 Text GLabel 3950 1950 2    50   Output ~ 0
 GND
-Text GLabel 4600 1800 0    50   Input ~ 0
+Text GLabel 4600 1900 0    50   Input ~ 0
 -12
-Text GLabel 4600 2000 0    50   Input ~ 0
+Text GLabel 4600 2450 0    50   Input ~ 0
 +12
 Text GLabel 5350 1900 0    50   Input ~ 0
 GND
 $Comp
-L Switch:SW_DPST ON/OFF1
+L Switch:SW_DPDT_x2 ON/OFF1
 U 1 1 5FEB7DE5
 P 4800 1900
-F 0 "ON/OFF1" H 4800 2225 50  0000 C CNN
-F 1 "SW_DPST" H 4800 2134 50  0000 C CNN
+F 0 "ON/OFF1" H 4800 2100 50  0000 C CNN
+F 1 "SW_DPST" H 4800 2200 50  0000 C CNN
 F 2 "RobsFoots:SW_CK_Lever_DPDT_72xx_CircularHoles" H 4800 1900 50  0001 C CNN
 F 3 "~" H 4800 1900 50  0001 C CNN
@@
 	1    0    0    -1
 $EndComp
-Wire Wire Line
-	5000 2000 5000 2350
 Wire Wire Line
 	5000 2350 5600 2350
@@
 Text Notes 7150 6750 0    157  ~ 0
 Schematic V0.0.1
+$Comp
+L Switch:SW_DPDT_x2 ON/OFF1
+U 2 1 5FEDA711
+P 4800 2450
+F 0 "ON/OFF1" H 4750 2250 50  0000 C CNN
+F 1 "SW_DPST" H 4750 2150 50  0000 C CNN
+F 2 "RobsFoots:SW_CK_Lever_DPDT_72xx_CircularHoles" H 4800 2450 50  0001 C CNN
+F 3 "~" H 4800 2450 50  0001 C CNN
+	2    4800 2450
+	1    0    0    -1
+$EndComp
+Text GLabel 7050 1850 0    50   Input ~ 0
+GND
+Text GLabel 7050 2650 0    50   Input ~ 0
+GND
+Text GLabel 8250 1850 0    50   Input ~ 0
+GND
+Text GLabel 8250 2650 0    50   Input ~ 0
+GND
+Text GLabel 9200 2650 0    50   Input ~ 0
+GND
+Text GLabel 9200 1850 0    50   Input ~ 0
+GND
 $EndSCHEMATC
