File: Front/Panel.kicad_pcb (KiCad board)
At the start: 2 copper layers, 68.3 x 200 mm, 28 parts, among them J1 INPUT POWER, J2 Conn_02x05_Odd_Even, J2 IN2, J3 Conn_02x05_Odd_Even, J4 Conn_02x05_Odd_Even, J5 Conn_02x05_Odd_Even, J6 Conn_02x05_Odd_Even, J7 Conn_02x05_Odd_Even

Commit message: New Mounting Holes
Parts:
- removed the J2 at (131.5, 43.6)
- removed the J2 at (92.7, 188.0)
- removed the J2 at (92.7, 170.0)
- removed the J2 at (92.7, 152.0)
- removed REF** (x6): MountingHole_3.2mm_M3_DIN965_Pad, MountingHole:MountingHole_3.2mm_M3_DIN965_Pad
- removed RV2 (x4): A100K, ROBSLIBRARY:Potentiometer-Panel
- added H1: MountingHole_Pad, MountingHole:MountingHole_3.2mm_M3_DIN965_Pad, F.Cu at (100.7, 215.2)
- added H1: MountingHole_Pad, MountingHole:MountingHole_3.2mm_M3_DIN965_Pad, F.Cu at (82.7, 215.2)
- added H1: MountingHole_Pad, MountingHole:MountingHole_3.2mm_M3_DIN965_Pad, F.Cu at (82.7, 22.2)
- added H1: MountingHole_Pad, MountingHole:MountingHole_3.2mm_M3_DIN965_Pad, F.Cu at (205.5, 124.2)
- added H1: MountingHole_Pad, MountingHole:MountingHole_3.2mm_M3_DIN965_Pad, F.Cu at (205.5, 55.7)
- added H1: MountingHole_Pad, MountingHole:MountingHole_3.2mm_M3_DIN965_Pad, F.Cu at (100.7, 22.2)
- added J2: Conn_02x05_Odd_Even, Connector_IDC:IDC-Header_2x05_P2.54mm_Vertical, F.Cu at (210.6, 134.6)
- moved J1 222.0 mm to (200.4, -17.9), turned to 90 degrees
- moved R2 198.5 mm to (214.5, -0.11), turned to 90 degrees
- moved R1 194.3 mm to (196.2, -4.68), turned to 270 degrees
- moved ON/OFF1 191.5 mm to (203.0, -1.13), turned to 0 degrees
- moved D2 189.9 mm to (213.0, 3.94), turned to 270 degrees
- moved D1 178.9 mm to (198.2, 3.94), turned to 270 degrees
- moved J3 159.9 mm to (210.6, 19.6), turned to 270 degrees
- moved J4 122.1 mm to (210.6, 42.6), turned to 270 degrees
- moved J5 92.0 mm to (210.6, 65.6), turned to 270 degrees
- moved J6 91.0 mm to (210.6, 111.6), turned to 270 degrees
- moved J7 79.1 mm to (210.6, 88.6), turned to 270 degrees
- moved G*** 75.2 mm to (28.7, 21.4)
- moved J2 47.9 mm to (52.7, 8.96)
- moved G*** 31.9 mm to (60.6, 29.2)
Routing:
- net (no net): track 722.7 -> 255.6 mm
Other:
- board size 68.3 x 200 mm -> 137.2 x 247.9 mm

Commit message: FP Boards Aligned
Parts:
- removed J1: INPUT POWER, Connector_IDC:IDC-Header_2x05_P2.54mm_Vertical
- removed J2, J3, J4, J5, J6, J7: Conn_02x05_Odd_Even, Connector_IDC:IDC-Header_2x05_P2.54mm_Vertical
- removed J2: IN2, ROBSLIBRARY:PANEL-LMNC
- removed R1, R2: 1K, Resistor_THT:R_Axial_DIN0204_L3.6mm_D1.6mm_P5.08mm_Horizontal
- D1, D2, ON/OFF1: moved to F.Cu
- H1 (x2): moved to B.Cu
- moved D2 142.2 mm to (84.2, 64.4)
- moved H1 128.9 mm to (91.7, 116.2)
- moved H1 128.8 mm to (91.7, 184.7)
- moved ON/OFF1 124.5 mm to (94.2, 59.4), turned to 180 degrees
- moved D1 116.3 mm to (99.0, 64.4)
Other:
- board size 137.2 x 247.9 mm -> 25 x 200 mm
- board text removed: "C H N 1"
- board text removed: "C H N 2"
- board text removed: "C H N 3"
- board text removed: "M A S T E R"

Commit message: FP Holes Added
Parts:
- removed ON/OFF1: SW_DPST, RobsFoots:SW_CK_Lever_DPDT_72xx_CircularHoles
- added SW9: RUNSTOP, RobsFoots:FP-MINITOGLE, F.Cu at (91.7, 54.7)
- D1, D2: footprint LED_THT:LED_D5.0mm -> RobsFoots:FP-LED_D5.0mm
- moved G*** 106.3 mm to (91.5, 131.0)
- moved G*** 87.6 mm to (90.8, 83.2)
Routing:
- net (no net): track 255.6 -> 0.00 mm
Other:
- outline, holes or cut-outs redrawn

Commit message: FP Labels
Parts:
- renumbered D2 to +12V, D1 to -12V
Other:
- board text added: "CLAYTUNE - BussBar V0.0.1 - By TwinTurbo"
- board text added: "OFF"
- board text added: "ON"
- board text removed: "CLAYTUNE - Simple Mixer V1.0 - By TwinTurbo"
- board text removed: "OUTPUT"
Changed lines of the file:
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@@
   (general
     (thickness 1.6)
-    (drawings 9)
+    (drawings 10)
     (tracks 0)
     (zones 0)
@@
       (effects (font (size 1 1) (thickness 0.15)))
     )
-    (fp_text value RUNSTOP (at 18.96 -11.51) (layer F.SilkS)
+    (fp_text value RUNSTOP (at 19.31 -7.25) (layer F.SilkS)
       (effects (font (size 1 1) (thickness 0.15)))
     )
@@
     (descr "LED, diameter 5.0mm, 2 pins, http://cdn-reichelt.de/documents/datenblatt/A500/LL-504BC2E-009.pdf")
     (tags "LED diameter 5.0mm 2 pins")
-    (fp_text reference D2 (at 1.27 -3.96 270) (layer F.SilkS)
-      (effects (font (size 1 1) (thickness 0.15)))
-    )
-    (fp_text value "LED +12" (at 1.27 3.96 270) (layer F.Fab)
+    (fp_text reference +12V (at 5.45 0.332) (layer F.SilkS)
+      (effects (font (size 1.5 1.5) (thickness 0.2)))
+    )
+    (fp_text value "LED +12" (at 1.13 8.122 270) (layer F.Fab)
       (effects (font (size 1 1) (thickness 0.15)))
     )
@@
     (descr "LED, diameter 5.0mm, 2 pins, http://cdn-reichelt.de/documents/datenblatt/A500/LL-504BC2E-009.pdf")
     (tags "LED diameter 5.0mm 2 pins")
-    (fp_text reference D1 (at 1.27 -3.96 270) (layer F.SilkS)
-      (effects (font (size 1 1) (thickness 0.15)))
-    )
-    (fp_text value "LED -12" (at 1.27 3.96 270) (layer F.Fab)
+    (fp_text reference -12V (at 5.41 0.624) (layer F.SilkS)
+      (effects (font (size 1.5 1.5) (thickness 0.2)))
+    )
+    (fp_text value "LED -12" (at 1.78 -11.996 270) (layer F.Fab)
       (effects (font (size 1 1) (thickness 0.15)))
     )
@@
   (module ROBSLIBRARY:GFX1FC (layer F.Cu)
     (at 90.8 83.17)
-    (fp_text reference G*** (at 0 0) (layer F.SilkS) hide
+    (fp_text reference G*** (at -25.43 -2.4) (layer F.SilkS) hide
       (effects (font (size 1.524 1.524) (thickness 0.3)))
     )
-    (fp_text value LOGO (at 0.75 0) (layer F.SilkS) hide
+    (fp_text value LOGO (at -17.46 -1.1) (layer F.SilkS) hide
       (effects (font (size 1.524 1.524) (thickness 0.3)))
     )
@@
       (xy -0.647259 -12.024255) (xy -0.626714 -12.016411)) (layer F.Cu) (width 0.01))
   )
+  (gr_text OFF (at 91.69 60.76) (layer F.SilkS)
+    (effects (font (size 2 1.5) (thickness 0.15)))
+  )
+  (gr_text ON (at 91.79 48.89) (layer F.SilkS)
+    (effects (font (size 2 1.5) (thickness 0.15)))
+  )
   (gr_text "For Kate\nBy \nTwinTurbo" (at 91.51 40.52) (layer B.Cu)
     (effects (font (size 2 2) (thickness 0.5)) (justify mirror))
-  )
-  (gr_text OUTPUT (at 67.96 38.68) (layer F.Cu)
-    (effects (font (size 1.5 1.5) (thickness 0.3) italic))
   )
   (gr_line (start 104.244 218.708) (end 104.244 18.708) (layer Edge.Cuts) (width 0.05))
@@
     (effects (font (size 3 3) (thickness 0.3) italic))
   )
-  (gr_text "CLAYTUNE - Simple Mixer V1.0 - By TwinTurbo" (at 102.604 127.058 90) (layer B.Cu)
+  (gr_text "CLAYTUNE - BussBar V0.0.1 - By TwinTurbo" (at 102.604 127.058 90) (layer B.Cu)
     (effects (font (size 1.5 1.5) (thickness 0.3) italic))
   )
