File: Front/Panel.kicad_pcb (KiCad board)
At the start: 2 copper layers, 25 x 200 mm, 11 parts, among them SW9 RUNSTOP

Commit message: Board/FP ready
Other:
- board text added: "BIG RED BUSS"
- board text added: "Big Red Buss- PCB V 0.1.0"
- board text added: "CLAYTUNE - Big Red Buss V0.1.0 - By TwinTurbo - JLCJLCJLCJLC"
- board text added: "CLAYTUNE Big Red Buss By TwinTurbo"
- board text removed: "CLAYTUNE - BussBar V0.0.1 - By TwinTurbo"
Changed lines of the file:
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@@
-(kicad_pcb (version 20171130) (host pcbnew "(5.1.7)-1")
+(kicad_pcb (version 20171130) (host pcbnew 5.1.5-52549c5~86~ubuntu18.04.1)
   (general
     (thickness 1.6)
-    (drawings 10)
+    (drawings 18)
     (tracks 0)
     (zones 0)
@@
       (xy -0.647259 -12.024255) (xy -0.626714 -12.016411)) (layer F.Cu) (width 0.01))
   )
+  (gr_text "Big Red Buss- PCB V 0.1.0" (at 231.42 173.66) (layer Dwgs.User)
+    (effects (font (size 4 4) (thickness 0.15)))
+  )
+  (gr_text CLAYTUNE (at 91.67 208.84) (layer F.Cu)
+    (effects (font (size 3 3) (thickness 0.3)))
+  )
+  (gr_line (start 79.204 98.43) (end 104.34 98.43) (layer F.SilkS) (width 1.5))
+  (gr_line (start 79.22 167.4) (end 104.356 167.4) (layer F.SilkS) (width 1.5))
+  (gr_line (start 79.074 129.13) (end 104.21 129.13) (layer F.SilkS) (width 1.5))
+  (gr_line (start 79.184 46.29) (end 104.32 46.29) (layer F.SilkS) (width 1.5))
+  (gr_line (start 79.16 28.75) (end 104.33 28.75) (layer F.SilkS) (width 1.5))
+  (gr_text "CLAYTUNE\nBig Red Buss\nBy TwinTurbo\n " (at 91.32 38.9) (layer F.SilkS)
+    (effects (font (size 2 2) (thickness 0.5)))
+  )
+  (gr_text "\nBIG\nRED\nBUSS\n\n " (at 91.41 156.47) (layer F.SilkS)
+    (effects (font (size 6 6) (thickness 1)))
+  )
   (gr_text OFF (at 91.69 60.76) (layer F.SilkS)
     (effects (font (size 2 1.5) (thickness 0.15)))
@@
     (effects (font (size 2 1.5) (thickness 0.15)))
   )
-  (gr_text "For Kate\nBy \nTwinTurbo" (at 91.51 40.52) (layer B.Cu)
+  (gr_text "For Kate\nBy \nTwinTurbo" (at 91.51 40.52) (layer B.SilkS)
     (effects (font (size 2 2) (thickness 0.5)) (justify mirror))
   )
@@
   (gr_circle (center 91.744 118.753) (end 91.758142 118.753) (layer F.Fab) (width 0.15))
   (gr_line (start 104.244 218.708) (end 79.244 218.708) (layer Edge.Cuts) (width 0.05))
-  (gr_text CLAYTUNE (at 91.71 209.76) (layer F.Cu)
-    (effects (font (size 3 3) (thickness 0.3) italic))
-  )
-  (gr_text "CLAYTUNE - BussBar V0.0.1 - By TwinTurbo" (at 102.604 127.058 90) (layer B.Cu)
+  (gr_text "CLAYTUNE - Big Red Buss V0.1.0 - By TwinTurbo   - JLCJLCJLCJLC" (at 102.604 127.058 90) (layer B.Cu)
     (effects (font (size 1.5 1.5) (thickness 0.3) italic))
   )
